File: BigMuffRipOff/BigMuffRipOff.kicad_sch (KiCad schematic)
At the start: 9 parts, among them J2 NMJ6HFD2, J3 NMJ6HFD2, J4 2125201004, J6 2125201004, J7 2125201004

Commit message: datasheet updates
womp womp
Changed lines of the file:
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@@
 	(wire
 		(pts
-			(xy 72.39 88.9) (xy 76.2 88.9)
+			(xy 64.77 85.09) (xy 76.2 85.09)
 		)
 		(stroke
@@
 	(wire
 		(pts
-			(xy 76.2 88.9) (xy 76.2 67.31)
+			(xy 76.2 85.09) (xy 76.2 67.31)
 		)
 		(stroke
@@
 	)
 	(sheet
-		(at 40.64 86.36)
+		(at 33.02 82.55)
 		(size 31.75 30.48)
 		(exclude_from_sim no)
@@
 		)
 		(property "Sheetname" "PowerStage"
-			(at 40.64 85.6484 0)
+			(at 33.02 81.8384 0)
 			(effects
 				(font
@@
 		)
 		(property "Sheetfile" "PowerStage.kicad_sch"
-			(at 40.64 117.4246 0)
+			(at 33.02 113.6146 0)
 			(effects
 				(font
@@
 		)
 		(property "Field2" ""
-			(at 40.64 86.36 0)
+			(at 33.02 82.55 0)
 			(effects
 				(font
@@
 		)
 		(pin "LDO_EN" input
-			(at 72.39 88.9 0)
-			(effects
-				(font
+			(at 64.77 85.09 0)
+			(effects
+				(font

Commit message: getting closer on finishing layout
Other:
- sheet Effect Stage ports: added SPI_MOSI; removed SPI_MISO
- sheet MCU ports: added SPI_MOSI; removed LDO_EN, SPI_MISO
Changed lines of the file:
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@@
 			)
 		)
-		(pin "SPI_MISO" input
-			(at 203.2 93.98 180)
+		(pin "CS_4" input
+			(at 203.2 109.22 180)
 			(effects
 				(font
@@
 			)
 		)
-		(pin "CS_4" input
-			(at 203.2 109.22 180)
+		(pin "SPI_MOSI" input
+			(at 203.2 93.98 180)
 			(effects
 				(font
@@
 		(pin "SPI_CLK" output
 			(at 182.88 90.17 0)
-			(effects
-				(font
-					(size 1.27 1.27)
-				)
-				(justify right)
-			)
-		)
-		(pin "SPI_MISO" output
-			(at 182.88 93.98 0)
 			(effects
 				(font
@@
 			)
 		)
-		(pin "LDO_EN" input
-			(at 149.86 88.9 180)
+		(pin "SPI_MOSI" output
+			(at 182.88 93.98 0)
 			(effects
 				(font
 					(size 1.27 1.27)
 				)
-				(justify left)
+				(justify right)
 			)
 		)
