File: BigMuffRipOff/EffectStage.kicad_sch (KiCad schematic)
At the start: 55 parts, among them Q1 BC549, Q2 BC549, Q3 BC549, Q4 BC549, U1 TPL0501-100DCNR, U2 TPL0501-100DCNR, U3 TPL0501-100DCNR, U5 TL071HIDBVR, U8 TPL0501-100DCNR

Commit message: starting to redo board layout
also finished changing the schematic
Parts:
- removed R28, R29: 30k, Resistor_SMD:R_0603_1608Metric, symbol Device:R
- added C21, C22: 0.1u, Capacitor_SMD:C_0603_1608Metric, symbol Device:C
- added U4, U7: TL071HIDBVR, 284867-E-footprint:SOT23_DBV_5_TEX, symbol TL071HIDBVR:TL071HIDBVR
- R23: value 5k -> 10k
- R24: value 10k -> 20k
Connections:
- net 4.5V: now also U3.2 (VDD), U8.2 (VDD); no longer U3.3 (GND), U8.3 (GND)
- net 9V: now also U4.5 (V+), U7.5 (V+); no longer U3.2 (VDD), U8.2 (VDD)
- net GND: now also U3.3 (GND), U3.7 (L), U8.3 (GND), U8.7 (L), U7.2 (V-)
- net at C18.1: now also U3.8 (H); no longer R23.1
- net at R23.2: now also R24.1, R25.1, U5.4 (IN-); no longer U3.1 (W)
- net at R24.2: now also U4.1 (OUT), U4.4 (IN-); no longer U8.1 (W)
- net at U8.8 (H): now also C13.1
- new net: C21.1, U8.1 (W)
- new net: R23.1, U7.1 (OUT), U7.4 (IN-)
- new net: C22.2, U7.3 (IN+)
- new net: C22.1, U3.1 (W)
- new net: C21.2, U4.3 (IN+)
- no-connect marks 2 -> 0
Other:
- moved on the sheet: C1, C10, C11, C12, C13, C17, C18, C2, C3, C4, C5, C6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

Commit message: did half of the changes
gonna finish the next have next time
Connections:
- net GND: now also U4.2 (V-)
- net SPI_MISO renamed SPI_MOSI
Changed lines of the file:
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@@
+	(wire
+		(pts
+			(xy 520.7 100.33) (xy 520.7 101.6)
+		)
+		(stroke
+			(width 0)
+			(type default)
+		)
+	)
 	(wire
 		(pts
@@
 		)
 	)
-	(hierarchical_label "SPI_MISO"
+	(hierarchical_label "SPI_MOSI"
 		(shape input)
 		(at 447.04 140.97 180)
@@
 		)
 	)
-	(hierarchical_label "SPI_MISO"
+	(hierarchical_label "SPI_MOSI"
 		(shape input)
 		(at 445.77 87.63 180)
@@
 		)
 	)
-	(hierarchical_label "SPI_MISO"
+	(hierarchical_label "SPI_MOSI"
 		(shape input)
 		(at 134.62 82.55 180)
@@
 		)
 	)
-	(hierarchical_label "SPI_MISO"
+	(hierarchical_label "SPI_MOSI"
 		(shape input)
 		(at 356.87 69.85 180)

Commit message: getting closer on finishing layout
Parts:
- added C23, C24, C25, C26: 0.1u, Capacitor_SMD:C_0603_1608Metric, symbol Device:C
Connections:
- net 4.5V: now also C23.1, C24.1, C25.1, C26.1
- net GND: now also C23.2, C24.2, C25.2, C26.2
Other:
- moved on the sheet: C2, C3
