File: BigMuffRipOff/EffectStage.kicad_sch (KiCad schematic)
At the start: 61 parts, among them Q1 BC549, Q2 BC549, Q3 BC549, Q4 BC549, U1 TPL0501-100DCNR, U2 TPL0501-100DCNR, U3 TPL0501-100DCNR, U4 TL071HIDBVR, U5 TL071HIDBVR, U7 TL071HIDBVR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

Commit message: no sure
Connections:
- net 4.5V: now also C21.2, C22.2, U4.3 (IN+), U7.3 (IN+)
Changed lines of the file:
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@@
 	)
 	(junction
-		(at 565.15 109.22)
+		(at 486.41 151.13)
 		(diameter 0)
 		(color 0 0 0 0)
 	)
 	(junction
-		(at 486.41 151.13)
+		(at 414.02 69.85)
 		(diameter 0)
 		(color 0 0 0 0)
 	)
 	(junction
-		(at 414.02 69.85)
+		(at 502.92 87.63)
 		(diameter 0)
 		(color 0 0 0 0)
@@
 	)
 	(junction
+		(at 502.92 140.97)
+		(diameter 0)
+		(color 0 0 0 0)
+	)
+	(junction
 		(at 232.41 82.55)
 		(diameter 0)
@@
 	)
 	(junction
-		(at 299.72 59.69)
+		(at 546.1 111.76)
 		(diameter 0)
 		(color 0 0 0 0)
 	)
 	(junction
-		(at 312.42 43.18)
+		(at 299.72 59.69)
 		(diameter 0)
 		(color 0 0 0 0)
 	)
 	(junction
-		(at 546.1 109.22)
+		(at 312.42 43.18)
 		(diameter 0)
 		(color 0 0 0 0)
@@
 	)
 	(junction
+		(at 565.15 111.76)
+		(diameter 0)
+		(color 0 0 0 0)
+	)
+	(junction
 		(at 229.87 43.18)
 		(diameter 0)
@@
 	(wire
 		(pts
-			(xy 546.1 109.22) (xy 565.15 109.22)
+			(xy 546.1 111.76) (xy 565.15 111.76)
 		)
 		(stroke
@@
 	(wire
 		(pts
+			(xy 502.92 87.63) (xy 509.27 87.63)
+		)
+		(stroke
+			(width 0)
+			(type default)
+		)
+	)
+	(wire
+		(pts
 			(xy 130.81 74.93) (xy 130.81 76.2)
 		)
@@
 	(wire
 		(pts
-			(xy 560.07 116.84) (xy 565.15 116.84)
+			(xy 502.92 135.89) (xy 502.92 140.97)
+		)
+		(stroke
+			(width 0)
+			(type default)
+		)
+	)
+	(wire
+		(pts
+			(xy 557.53 120.65) (xy 561.34 120.65)
 		)
 		(stroke
@@
 	(wire
 		(pts
-			(xy 546.1 102.87) (xy 546.1 109.22)
+			(xy 546.1 102.87) (xy 546.1 111.76)
 		)
 		(stroke
@@
 	(wire
 		(pts
-			(xy 499.11 140.97) (xy 509.27 140.97)
+			(xy 499.11 140.97) (xy 502.92 140.97)
 		)
 		(stroke
@@
 	(wire
 		(pts
+			(xy 561.34 120.65) (xy 561.34 116.84)
+		)
+		(stroke
+			(width 0)
+			(type default)
+		)
+	)
+	(wire
+		(pts
 			(xy 220.98 43.18) (xy 217.17 43.18)
 		)
@@
 	(wire
 		(pts
+			(xy 546.1 111.76) (xy 546.1 121.92)
+		)
+		(stroke
+			(width 0)
+			(type default)
+		)
+	)
+	(wire
+		(pts
 			(xy 391.16 69.85) (xy 400.05 69.85)
 		)
@@
 	(wire
 		(pts
+			(xy 502.92 140.97) (xy 509.27 140.97)
+		)
+		(stroke
+			(width 0)
+			(type default)
+		)
+	)
+	(wire
+		(pts
 			(xy 486.41 85.09) (xy 482.6 85.09)
 		)
@@
 	(wire
 		(pts
+			(xy 502.92 82.55) (xy 502.92 87.63)
+		)
+		(stroke
+			(width 0)
+			(type default)
+		)
+	)
+	(wire
+		(pts
 			(xy 443.23 80.01) (xy 443.23 81.28)
 		)
@@
 	(wire
 		(pts
-			(xy 499.11 87.63) (xy 509.27 87.63)
+			(xy 499.11 87.63) (xy 502.92 87.63)
 		)
 		(stroke
@@
 	(wire
 		(pts
-			(xy 565.15 109.22) (xy 565.15 111.76)
-		)
-		(stroke
-			(width 0)
-			(type default)
-		)
-	)
-	(wire
-		(pts
 			(xy 443.23 71.12) (xy 452.12 71.12)
 		)
@@
 	(wire
 		(pts
-			(xy 546.1 109.22) (xy 546.1 121.92)
+			(xy 335.28 69.85) (xy 335.28 77.47)
 		)
 		(stroke
@@
 	(wire
 		(pts
-			(xy 335.28 69.85) (xy 335.28 77.47)
+			(xy 118.11 97.79) (xy 118.11 105.41)
 		)
 		(stroke
@@
 	(wire
 		(pts
-			(xy 118.11 97.79) (xy 118.11 105.41)
+			(xy 299.72 59.69) (xy 309.88 59.69)
 		)
 		(stroke
@@
 	(wire
 		(pts
-			(xy 299.72 59.69) (xy 309.88 59.69)
+			(xy 118.11 77.47) (xy 118.11 87.63)
 		)
 		(stroke
@@
 	(wire
 		(pts
-			(xy 118.11 77.47) (xy 118.11 87.63)
+			(xy 101.6 77.47) (xy 96.52 77.47)
 		)
 		(stroke
@@
 	(wire
 		(pts
-			(xy 101.6 77.47) (xy 96.52 77.47)
+			(xy 335.28 31.75) (xy 335.28 43.18)
 		)
 		(stroke
@@
 	(wire
 		(pts
-			(xy 335.28 31.75) (xy 335.28 43.18)
+			(xy 561.34 116.84) (xy 565.15 116.84)
 		)
 		(stroke
@@
 	(wire
 		(pts
-			(xy 565.15 109.22) (xy 565.15 90.17)
+			(xy 565.15 90.17) (xy 565.15 111.76)
 		)
 		(stroke
@@
 	)
 	(symbol
+		(lib_id "power:VCC")
+		(at 502.92 135.89 0)
+		(unit 1)
+		(exclude_from_sim no)
+		(in_bom yes)
+		(on_board yes)
+		(dnp no)
+		(fields_autoplaced yes)
+		(property "Reference" "#PWR055"
+			(at 502.92 139.7 0)
+			(effects
+				(font
+					(size 1.27 1.27)
+				)
+				(hide yes)
+			)
+		)
+		(property "Value" "4.5V"
+			(at 502.92 130.81 0)
+			(effects
+				(font
+					(size 1.27 1.27)
+				)
+			)
+		)
+		(property "Footprint" ""
+			(at 502.92 135.89 0)
+			(effects
+				(font
+					(size 1.27 1.27)
+				)
+				(hide yes)
+			)
+		)
+		(property "Datasheet" ""
+			(at 502.92 135.89 0)
+			(effects
+				(font
+					(size 1.27 1.27)
+				)
+				(hide yes)
+			)
+		)
+		(property "Description" "Power symbol creates a global label with name \"VCC\""
+			(at 502.92 135.89 0)
+			(effects
+				(font
+					(size 1.27 1.27)
+				)
+				(hide yes)
+			)
+		)
+		(pin "1"
+		)
+		(instances
+			(project "BigMuffRipOff"
+				(path "/ee7a6669-1f80-4e5e-942b-cae2c32afcf3/cc61f787-c881-4bf8-bc84-97b283f90893"
+					(reference "#PWR055")
+					(unit 1)
+				)
+			)
+		)
+	)
+	(symbol
 		(lib_id "Transistor_BJT:BC549")
 		(at 250.19 82.55 0)
@@
 	(symbol
 		(lib_id "power:VCC")
-		(at 560.07 116.84 0)
+		(at 557.53 120.65 0)
 		(unit 1)
 		(exclude_from_sim no)
@@
 		(fields_autoplaced yes)
 		(property "Reference" "#PWR032"
-			(at 560.07 120.65 0)
+			(at 557.53 124.46 0)
 			(effects
 				(font
@@
 		)
 		(property "Value" "4.5V"
-			(at 560.07 111.76 0)
+			(at 557.53 115.57 0)
 			(effects
 				(font
@@
 		)
 		(property "Footprint" ""
-			(at 560.07 116.84 0)
+			(at 557.53 120.65 0)
 			(effects
 				(font
@@
 		)
 		(property "Datasheet" ""
-			(at 560.07 116.84 0)
+			(at 557.53 120.65 0)
 			(effects
 				(font
@@
 		)
 		(property "Description" "Power symbol creates a global label with name \"VCC\""
-			(at 560.07 116.84 0)
+			(at 557.53 120.65 0)
 			(effects
 				(font
@@
 					(unit 1)
 				)
+			)
+		)
+	)
+	(symbol
+		(lib_id "power:VCC")
+		(at 502.92 82.55 0)
+		(unit 1)
+		(exclude_from_sim no)
+		(in_bom yes)
+		(on_board yes)
+		(dnp no)
+		(fields_autoplaced yes)
+		(property "Reference" "#PWR056"
+			(at 502.92 86.36 0)
+			(effects
+				(font
+					(size 1.27 1.27)
+				)
+				(hide yes)
+			)
+		)
+		(property "Value" "4.5V"
+			(at 502.92 77.47 0)
+			(effects
+				(font
+					(size 1.27 1.27)
+				)
+			)
+		)
+		(property "Footprint" ""
+			(at 502.92 82.55 0)
+			(effects
+				(font
+					(size 1.27 1.27)
+				)
+				(hide yes)
+			)
+		)
+		(property "Datasheet" ""
+			(at 502.92 82.55 0)
+			(effects
+				(font
+					(size 1.27 1.27)
+				)
+				(hide yes)
+			)
+		)
+		(property "Description" "Power symbol creates a global label with name \"VCC\""
+			(at 502.92 82.55 0)
+			(effects
+				(font
+					(size 1.27 1.27)
+				)
+				(hide yes)
+			)
+		)
+		(pin "1"
+		)
+		(instances
+			(project "BigMuffRipOff"
+				(path "/ee7a6669-1f80-4e5e-942b-cae2c32afcf3/cc61f787-c881-4bf8-bc84-97b283f90893"
+					(reference "#PWR056")
+					(unit 1)
+				)

Commit message: look mom i did it
the board is done
Parts:
- added R26, R27, R28: 500k, Resistor_SMD:R_0603_1608Metric, symbol Device:R
Connections:
- net 4.5V: now also R26.1, R27.1, R28.2; no longer C21.2, C22.2, U4.3 (IN+), U5.3 (IN+), U7.3 (IN+)
- new net: C22.2, R26.2, U7.3 (IN+)
- new net: R28.1, U5.3 (IN+)
- new net: C21.2, R27.2, U4.3 (IN+)
