File: BigMuffRipOff/MCU.kicad_sch (KiCad schematic)
At the start: 6 parts, among them J1 284697-E, SW3 B3FS-1010P, U9 STM8L152K4T6

Commit message: did half of the changes
gonna finish the next have next time
Connections:
- net SPI_MISO is gone; now on net CS_1: U9.14 (PB1)
- net CS_1: no longer U9.18 (PB5)
- net CS_2: now also U9.16 (PB3); no longer U9.17 (PB4)
- net CS_3: now also U9.17 (PB4); no longer U9.16 (PB3)
- net SPI_CLK: now also U9.18 (PB5); no longer U9.13 (PB0)
- net SPI_MOSI: now reaches U9.19 (PB6)
Changed lines of the file:
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@@
+	)
+	(no_connect
+		(at 69.85 72.39)
 	)
 	(no_connect
@@
 	)
 	(no_connect
+		(at 69.85 90.17)
+	)
+	(no_connect
 		(at 146.05 62.23)
 	)
@@
 	)
 	(no_connect
-		(at 69.85 90.17)
-	)
-	(no_connect
 		(at 146.05 64.77)
 	)
@@
 	)
 	(no_connect
-		(at 69.85 87.63)
-	)
-	(no_connect
 		(at 69.85 57.15)
 	)
@@
 	(wire
 		(pts
+			(xy 64.77 77.47) (xy 69.85 77.47)
+		)
+		(stroke
+			(width 0)
+			(type default)
+		)
+	)
+	(wire
+		(pts
 			(xy 66.04 127) (xy 40.64 127)
 		)
@@
 	(wire
 		(pts
+			(xy 64.77 74.93) (xy 69.85 74.93)
+		)
+		(stroke
+			(width 0)
+			(type default)
+		)
+	)
+	(wire
+		(pts
 			(xy 148.59 85.09) (xy 146.05 85.09)
 		)
@@
 	(wire
 		(pts
+			(xy 64.77 82.55) (xy 69.85 82.55)
+		)
+		(stroke
+			(width 0)
+			(type default)
+		)
+	)
+	(wire
+		(pts
 			(xy 38.1 54.61) (xy 38.1 59.69)
 		)
@@
 	(wire
 		(pts
-			(xy 64.77 72.39) (xy 69.85 72.39)
-		)
-		(stroke
-			(width 0)
-			(type default)
-		)
-	)
-	(wire
-		(pts
 			(xy 66.04 113.03) (xy 66.04 115.57)
 		)
@@
 	(wire
 		(pts
+			(xy 64.77 87.63) (xy 69.85 87.63)
+		)
+		(stroke
+			(width 0)
+			(type default)
+		)
+	)
+	(wire
+		(pts
+			(xy 64.77 85.09) (xy 69.85 85.09)
+		)
+		(stroke
+			(width 0)
+			(type default)
+		)
+	)
+	(wire
+		(pts
+			(xy 40.64 115.57) (xy 40.64 118.11)
+		)
+		(stroke
+			(width 0)
+			(type default)
+		)
+	)
+	(wire
+		(pts
+			(xy 53.34 31.75) (xy 53.34 34.29)
+		)
+		(stroke
+			(width 0)
+			(type default)
+		)
+	)
+	(wire
+		(pts
+			(xy 165.1 25.4) (xy 165.1 26.67)
+		)
+		(stroke
+			(width 0)
+			(type default)
+		)
+	)
+	(wire
+		(pts
+			(xy 66.04 107.95) (xy 66.04 110.49)
+		)
+		(stroke
+			(width 0)
+			(type default)
+		)
+	)
+	(wire
+		(pts
+			(xy 170.18 25.4) (xy 170.18 26.67)
+		)
+		(stroke
+			(width 0)
+			(type default)
+		)
+	)
+	(wire
+		(pts
+			(xy 36.83 115.57) (xy 40.64 115.57)
+		)
+		(stroke
+			(width 0)
+			(type default)
+		)
+	)
+	(wire
+		(pts
+			(xy 165.1 49.53) (xy 165.1 52.07)
+		)
+		(stroke
+			(width 0)
+			(type default)
+		)
+	)
+	(wire
+		(pts
+			(xy 148.59 82.55) (xy 146.05 82.55)
+		)
+		(stroke
+			(width 0)
+			(type default)
+		)
+	)
+	(wire
+		(pts
+			(xy 40.64 115.57) (xy 43.18 115.57)
+		)
+		(stroke
+			(width 0)
+			(type default)
+		)
+	)
+	(wire
+		(pts
+			(xy 66.04 115.57) (xy 66.04 127)
+		)
+		(stroke
+			(width 0)
+			(type default)
+		)
+	)
+	(wire
+		(pts
+			(xy 43.18 110.49) (xy 36.83 110.49)
+		)
+		(stroke
+			(width 0)
+			(type default)
+		)
+	)
+	(wire
+		(pts
+			(xy 38.1 54.61) (xy 40.64 54.61)
+		)
+		(stroke
+			(width 0)
+			(type default)
+		)
+	)
+	(wire
+		(pts
+			(xy 66.04 110.49) (xy 66.04 113.03)
+		)
+		(stroke
+			(width 0)
+			(type default)
+		)
+	)
+	(wire
+		(pts
 			(xy 64.77 80.01) (xy 69.85 80.01)
 		)
@@
 	(wire
 		(pts
-			(xy 40.64 115.57) (xy 40.64 118.11)
-		)
-		(stroke
-			(width 0)
-			(type default)
-		)
-	)
-	(wire
-		(pts
-			(xy 53.34 31.75) (xy 53.34 34.29)
-		)
-		(stroke
-			(width 0)
-			(type default)
-		)
-	)
-	(wire
-		(pts
-			(xy 165.1 25.4) (xy 165.1 26.67)
-		)
-		(stroke
-			(width 0)
-			(type default)
-		)
-	)
-	(wire
-		(pts
-			(xy 66.04 107.95) (xy 66.04 110.49)
-		)
-		(stroke
-			(width 0)
-			(type default)
-		)
-	)
-	(wire
-		(pts
-			(xy 170.18 25.4) (xy 170.18 26.67)
-		)
-		(stroke
-			(width 0)
-			(type default)
-		)
-	)
-	(wire
-		(pts
-			(xy 36.83 115.57) (xy 40.64 115.57)
-		)
-		(stroke
-			(width 0)
-			(type default)
-		)
-	)
-	(wire
-		(pts
-			(xy 165.1 49.53) (xy 165.1 52.07)
-		)
-		(stroke
-			(width 0)
-			(type default)
-		)
-	)
-	(wire
-		(pts
-			(xy 148.59 82.55) (xy 146.05 82.55)
-		)
-		(stroke
-			(width 0)
-			(type default)
-		)
-	)
-	(wire
-		(pts
-			(xy 40.64 115.57) (xy 43.18 115.57)
-		)
-		(stroke
-			(width 0)
-			(type default)
-		)
-	)
-	(wire
-		(pts
-			(xy 64.77 77.47) (xy 69.85 77.47)
-		)
-		(stroke
-			(width 0)
-			(type default)
-		)
-	)
-	(wire
-		(pts
-			(xy 64.77 82.55) (xy 69.85 82.55)
-		)
-		(stroke
-			(width 0)
-			(type default)
-		)
-	)
-	(wire
-		(pts
-			(xy 66.04 115.57) (xy 66.04 127)
-		)
-		(stroke
-			(width 0)
-			(type default)
-		)
-	)
-	(wire
-		(pts
-			(xy 43.18 110.49) (xy 36.83 110.49)
-		)
-		(stroke
-			(width 0)
-			(type default)
-		)
-	)
-	(wire
-		(pts
-			(xy 38.1 54.61) (xy 40.64 54.61)
-		)
-		(stroke
-			(width 0)
-			(type default)
-		)
-	)
-	(wire
-		(pts
-			(xy 66.04 110.49) (xy 66.04 113.03)
-		)
-		(stroke
-			(width 0)
-			(type default)
-		)
-	)
-	(wire
-		(pts
-			(xy 64.77 74.93) (xy 69.85 74.93)
-		)
-		(stroke
-			(width 0)
-			(type default)
-		)
-	)
-	(wire
-		(pts
 			(xy 50.8 54.61) (xy 69.85 54.61)
 		)
@@
 		(pts
 			(xy 36.83 113.03) (xy 43.18 113.03)
-		)
-		(stroke
-			(width 0)
-			(type default)
-		)
-	)
-	(wire
-		(pts
-			(xy 64.77 85.09) (xy 69.85 85.09)
 		)
 		(stroke
@@
 	(hierarchical_label "SPI_CLK"
 		(shape output)
-		(at 64.77 72.39 180)
+		(at 64.77 85.09 180)
 		(effects
 			(font
@@
 	(hierarchical_label "CS_1"
 		(shape output)
-		(at 64.77 85.09 180)
+		(at 64.77 74.93 180)
 		(effects
 			(font
@@
 		)
 	)
-	(hierarchical_label "SPI_MISO"
-		(shape output)
-		(at 64.77 74.93 180)
+	(hierarchical_label "SPI_MOSI"
+		(shape output)
+		(at 64.77 87.63 180)
 		(effects
 			(font
@@
 	(hierarchical_label "CS_2"
 		(shape output)
+		(at 64.77 80.01 180)
+		(effects
+			(font
+				(size 1.27 1.27)
+			)
+			(justify right)
+		)
+	)
+	(hierarchical_label "CS_3"
+		(shape output)
 		(at 64.77 82.55 180)
 		(effects
 			(font
-				(size 1.27 1.27)
-			)
-			(justify right)
-		)
-	)
-	(hierarchical_label "CS_3"
-		(shape output)
-		(at 64.77 80.01 180)
-		(effects
-			(font

Commit message: getting closer on finishing layout
Connections:
- net LDO_EN is gone; now on net Pot_2: U9.5 (PA5)
- net CS_1: now also U9.20 (PB7); no longer U9.14 (PB1)
- net CS_2: now also U9.23 (PD6); no longer U9.16 (PB3)
- net CS_3: now also U9.22 (PD5); no longer U9.17 (PB4)
- net CS_4: now also U9.21 (PD4); no longer U9.15 (PB2)
- net Pot_1: now also U9.4 (PA4); no longer U9.22 (PD5)
- net Pot_2: no longer U9.23 (PD6)
- net Pot_3: now also U9.6 (PA6); no longer U9.24 (PD7)
- no-connect marks 18 -> 19
Changed lines of the file:
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@@
-	)
-	(no_connect
-		(at 69.85 62.23)
-	)
-	(no_connect
-		(at 146.05 80.01)
 	)
 	(no_connect
@@
 	)
 	(no_connect
-		(at 69.85 67.31)
-	)
-	(no_connect
 		(at 146.05 77.47)
 	)
@@
 	)
 	(no_connect
+		(at 69.85 77.47)
+	)
+	(no_connect
+		(at 69.85 80.01)
+	)
+	(no_connect
 		(at 146.05 72.39)
 	)
 	(no_connect
+		(at 146.05 87.63)
+	)
+	(no_connect
 		(at 69.85 59.69)
 	)
 	(no_connect
-		(at 69.85 90.17)
-	)
-	(no_connect
 		(at 146.05 62.23)
 	)
@@
 	)
 	(no_connect
+		(at 69.85 82.55)
+	)
+	(no_connect
 		(at 146.05 64.77)
 	)
 	(no_connect
+		(at 69.85 74.93)
+	)
+	(no_connect
 		(at 146.05 52.07)
 	)
@@
 	(wire
 		(pts
-			(xy 64.77 77.47) (xy 69.85 77.47)
+			(xy 67.31 62.23) (xy 69.85 62.23)
+		)
+		(stroke
+			(width 0)
+			(type default)
+		)
+	)
+	(wire
+		(pts
+			(xy 146.05 85.09) (xy 149.86 85.09)
 		)
 		(stroke
@@
 	(wire
 		(pts
-			(xy 64.77 74.93) (xy 69.85 74.93)
-		)
-		(stroke
-			(width 0)
-			(type default)
-		)
-	)
-	(wire
-		(pts
-			(xy 148.59 85.09) (xy 146.05 85.09)
-		)
-		(stroke
-			(width 0)
-			(type default)
-		)
-	)
-	(wire
-		(pts
-			(xy 64.77 82.55) (xy 69.85 82.55)
-		)
-		(stroke
-			(width 0)
-			(type default)
-		)
-	)
-	(wire
-		(pts
 			(xy 38.1 54.61) (xy 38.1 59.69)
 		)
@@
 	(wire
 		(pts
+			(xy 67.31 67.31) (xy 69.85 67.31)
+		)
+		(stroke
+			(width 0)
+			(type default)
+		)
+	)
+	(wire
+		(pts
 			(xy 66.04 113.03) (xy 66.04 115.57)
 		)
@@
 	(wire
 		(pts
+			(xy 64.77 90.17) (xy 69.85 90.17)
+		)
+		(stroke
+			(width 0)
+			(type default)
+		)
+	)
+	(wire
+		(pts
 			(xy 40.64 115.57) (xy 40.64 118.11)
 		)
@@
 	(wire
 		(pts
-			(xy 148.59 82.55) (xy 146.05 82.55)
-		)
-		(stroke
-			(width 0)
-			(type default)
-		)
-	)
-	(wire
-		(pts
 			(xy 40.64 115.57) (xy 43.18 115.57)
 		)
@@
 	(wire
 		(pts
+			(xy 146.05 82.55) (xy 149.86 82.55)
+		)
+		(stroke
+			(width 0)
+			(type default)
+		)
+	)
+	(wire
+		(pts
 			(xy 66.04 115.57) (xy 66.04 127)
 		)
@@
 	(wire
 		(pts
+			(xy 67.31 64.77) (xy 69.85 64.77)
+		)
+		(stroke
+			(width 0)
+			(type default)
+		)
+	)
+	(wire
+		(pts
 			(xy 66.04 110.49) (xy 66.04 113.03)
 		)
@@
 	(wire
 		(pts
-			(xy 64.77 80.01) (xy 69.85 80.01)
-		)
-		(stroke
-			(width 0)
-			(type default)
-		)
-	)
-	(wire
-		(pts
 			(xy 50.8 54.61) (xy 69.85 54.61)
 		)
@@
 	(wire
 		(pts
-			(xy 69.85 64.77) (xy 66.04 64.77)
-		)
-		(stroke
-			(width 0)
-			(type default)
-		)
-	)
-	(wire
-		(pts
-			(xy 148.59 87.63) (xy 146.05 87.63)
+			(xy 146.05 80.01) (xy 149.86 80.01)
 		)
 		(stroke
@@
 	(hierarchical_label "CS_1"
 		(shape output)
-		(at 64.77 74.93 180)
+		(at 64.77 90.17 180)
 		(effects
 			(font
@@
 	(hierarchical_label "CS_4"
 		(shape output)
-		(at 64.77 77.47 180)
-		(effects
-			(font
-				(size 1.27 1.27)
-			)
-			(justify right)
+		(at 149.86 80.01 0)
+		(effects
+			(font
+				(size 1.27 1.27)
+			)
+			(justify left)
 		)
 	)
@@
 	(hierarchical_label "CS_2"
 		(shape output)
-		(at 64.77 80.01 180)
-		(effects
-			(font
-				(size 1.27 1.27)
-			)
-			(justify right)
+		(at 149.86 85.09 0)
+		(effects
+			(font
+				(size 1.27 1.27)
+			)
+			(justify left)
 		)
 	)
 	(hierarchical_label "CS_3"
 		(shape output)
-		(at 64.77 82.55 180)
-		(effects
-			(font
-				(size 1.27 1.27)
-			)
-			(justify right)
+		(at 149.86 82.55 0)
+		(effects
+			(font
+				(size 1.27 1.27)
+			)
+			(justify left)
 		)
 	)
 	(hierarchical_label "Pot_1"
 		(shape input)
-		(at 148.59 82.55 0)
-		(effects
-			(font
-				(size 1.27 1.27)
-			)
-			(justify left)
+		(at 67.31 62.23 180)
+		(effects
+			(font
+				(size 1.27 1.27)
+			)
+			(justify right)
 		)
 	)
 	(hierarchical_label "Pot_3"
 		(shape input)
-		(at 148.59 87.63 0)
-		(effects
-			(font
-				(size 1.27 1.27)
-			)
-			(justify left)
+		(at 67.31 67.31 180)
+		(effects
+			(font
+				(size 1.27 1.27)
+			)
+			(justify right)
 		)
 	)
 	(hierarchical_label "Pot_2"
 		(shape input)
-		(at 148.59 85.09 0)
-		(effects
-			(font
-				(size 1.27 1.27)
-			)
-			(justify left)
-		)
-	)
-	(hierarchical_label "LDO_EN"
-		(shape output)
-		(at 66.04 64.77 180)
-		(effects
-			(font
+		(at 67.31 64.77 180)
+		(effects
+			(font

Commit message: please dont break plsplspls
Parts:
- added C27: 10n, Capacitor_SMD:C_0603_1608Metric, symbol Device:C
- added C28: 100n, Capacitor_SMD:C_0603_1608Metric, symbol Device:C
- added C30: 1u, Capacitor_SMD:C_0603_1608Metric, symbol Device:C
- added J8: Conn_01x04, Connector_PinHeader_2.54mm:PinHeader_1x04_P2.54mm_Vertical, symbol Connector_Generic:Conn_01x04
Connections:
- net 3.3V: now also U9.9 (VLCD), C27.1, C28.1, C30.2
- net GND: now also C27.2, C28.2, C30.1, J8.3 (Pin_3), J8.4 (Pin_4)
- net UART_RX: now reaches U9.27 (PC2)
- net UART_RX: now also J8.1 (Pin_1)
- net UART_TX: now reaches U9.28 (PC3)
- net UART_TX: now also J8.2 (Pin_2)
- no-connect marks 19 -> 16
