File: Overdrive/Overdrive/Overdrive.kicad_sch (KiCad schematic)
At the start: 0 parts

Commit message: finished Overdrive schematic
Parts:
- added C1, C2: 4.7u, Capacitor_SMD:C_0603_1608Metric_Pad1.08x0.95mm_HandSolder, symbol Device:C
- added C3: 0.1u, Capacitor_SMD:C_0603_1608Metric, symbol Device:C
- added C4, C7: 22u, Capacitor_SMD:C_0603_1608Metric, symbol Device:C
- added C5: 100u, Capacitor_SMD:C_1206_3216Metric, symbol Device:C
- added C6: 1u, Capacitor_SMD:C_0603_1608Metric, symbol Device:C
- added C8: 0.3u, Capacitor_SMD:C_0603_1608Metric, symbol Device:C
- added D1, D2, D3, D4, D5: 1N4148, Diode_THT:D_DO-35_SOD27_P7.62mm_Horizontal, symbol Diode:1N4148
- added J1: Conn_02x08_Counter_Clockwise, Connector_PinHeader_1.00mm:PinHeader_2x08_P1.00mm_Horizontal, symbol Connector_Generic:Conn_02x08_Counter_Clockwise
- added Q1, Q2: 2N3904, Package_TO_SOT_THT:TO-92_Inline, symbol Transistor_BJT:2N3904
- added R1, R2, R5: 10k, Resistor_SMD:R_0603_1608Metric, symbol Device:R
- added R10, R4: 1k, Resistor_SMD:R_0603_1608Metric, symbol Device:R
- added R11: 40k, Resistor_SMD:R_0603_1608Metric, symbol Device:R
- added R12: 36k, Resistor_SMD:R_0603_1608Metric, symbol Device:R
- added R13: 6.2k, Resistor_SMD:R_0603_1608Metric, symbol Device:R
- added R14: 9k, Resistor_SMD:R_0603_1608Metric, symbol Device:R
- added R3: 1M, Resistor_SMD:R_0603_1608Metric, symbol Device:R
- added R6: 100k, Resistor_SMD:R_0603_1608Metric, symbol Device:R
- added R7: 130k, Resistor_SMD:R_0603_1608Metric, symbol Device:R
- added R8: 18k, Resistor_SMD:R_0603_1608Metric, symbol Device:R
- added R9: 100, Resistor_SMD:R_0603_1608Metric, symbol Device:R
- added U1: RTB05W, Converter_DCDC:Converter_DCDC_RECOM_R-78B-2.0_THT, symbol Regulator_Switching:R-78B1.5-2.0
- added U2: AD5160, Package_TO_SOT_SMD:SOT-23-8, symbol Potentiometer_Digital:AD5160
- added U3, U4: TL071, symbol Amplifier_Operational:TL071
- added U5: AD8400ARZ1, R_8_ADI, symbol AD8400ARZ1:AD8400ARZ1
Connections:
- new net: C8.1, D5.2 (A)
- new net: C7.2, C8.2, D1.1 (K), R14.2
- new net: C3.1, U2.1 (W)
- new net: C3.2, R5.1
- new net: C7.1, Q2.3 (C), R13.1
- new net: R4.1, U2.7 (B)
- new net: R5.2, R6.2, U3.2 (-)
- new net: C5.2, R10.2, R9.1
- new net: Q1.1 (E), R9.2
- new net: D4.2 (A), D5.1 (K)
- new net: C4.1, U4.2 (-), U4.6
- new net: C4.2, Q1.2 (B), R7.1, R8.2
- new net: D1.2 (A), D2.1 (K)
- new net: D2.2 (A), D3.1 (K)
- new net: D3.2 (A), D4.1 (K)
- new net: R6.1, U3.6, U4.3 (+)
- new net: R3.1, U3.3 (+)
- new net: R1.2, R2.1, R3.2
- new net: C6.2, Q2.2 (B), R11.1, R12.2
- new net: R14.1, U5.8 (A1)
- new net: Q1.3 (C), Q2.1 (E)
- new net 12V: C1.1, J1.1 (Pin_1), J1.16 (Pin_16), R1.1, R11.2, R13.2, R7.2, U1.1 (IN), U3.7 (V+), U4.7 (V+), U5.6 (VDD)
- new net 3.3V: C2.1, U1.3 (OUT), U2.2 (V_{DD})
- new net CS0: J1.6 (Pin_6), U2.6 (~{CS})
- new net CS1: J1.4 (Pin_4), U5.3 (CS*)
- new net GND: C1.2, C2.2, C5.1, C6.1, J1.10 (Pin_10), J1.15 (Pin_15), J1.2 (Pin_2), J1.7 (Pin_7), R10.1, R12.1, R2.2, R4.2, R8.1, U1.2 (GND), U2.3 (GND), U3.4 (V-), U4.4 (V-), U5.1 (B1), U5.2 (GND)
- new net GUITAR_IN: J1.13 (Pin_13), U2.8 (A)
- new net GUITAR_OUT: J1.12 (Pin_12), U5.7 (W1)
- new net MOSI: J1.11 (Pin_11), U2.5 (SDI), U5.4 (SDI)
- new net SPI_CLK: J1.14 (Pin_14), U2.4 (CLK), U5.5 (CLK)
- no-connect marks 0 -> 8
Other:
- note added: "12 to 3.3 Converter"
- note added: "Connector to Analog Controller"
- note added: "KiCad Power Flags for ERC"
- note added: "Overdrive Pedal"
- note added: "This resistor is 9.0k instead of 9.5k on the hand-drawn schematic because there are no digital 500 ohm pots only 1k digital pots"
- company: (none) -> RGA
- title: (none) -> Overdrive
