File: BigMuffRipOff/New Big Muff/PowerStage.kicad_sch (KiCad schematic)
At the start: 7 parts, among them J5 PJ-007, U10 R-78E3.3-0.5, U6 ADP7118AUJZ-4.5-R7

Commit message: new big muff completed
Parts:
- removed J5: PJ-007, 284867-E-footprint:CONN_PJ-007_SSD, symbol PJ-007:PJ-007
- removed U10: R-78E3.3-0.5, Converter_DCDC:Converter_DCDC_RECOM_R-78E-0.5_THT, symbol Regulator_Switching:R-78E3.3-0.5
- added U10: LM2940IMP-9.0/NOPB, GTSR_KiCAD_Footprints:DCY0004A_N, symbol LDO:LM2940IMP-9.0_NOPB
- C14: value 10u -> 22u
- C15: value 10u -> 0.47u
Connections:
- net 9V: now also U10.3 (OUT)
- net GND: now also U10.2 (GND), U10.4 (GND)
- net 3.3V renamed 12V
- net 12V: now also U10.1 (IN)
Other:
- moved on the sheet: C19, C20, U6
