File: BigMuffRipOff/New Big Muff/BigMuffRipOff.kicad_pcb (KiCad board)
At the start: 4 copper layers, 60.9 x 32 mm, 78 parts, among them J1 Conn_02x08_Odd_Even, Q1 BC549, Q2 BC549, Q3 BC549, Q4 BC549, U1 TPL0501-100DCNR, U10 LM2940IMP-9.0/NOPB, U2 TPL0501-100DCNR, U3 TPL0501-100DCNR, U4 TL071HIDBVR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

Commit message: made changes for power
Parts:
- moved C19 3.18 mm to (133.4, 73.8), turned to 90 degrees
- moved U6 1.80 mm to (130.0, 77.0)
- moved R29 1.63 mm to (126.4, 94.0)
- moved C20 1.40 mm to (133.6, 78.8)
- moved C16 1.02 mm to (129.2, 94.8)
Routing:
- net 4.5V: track 39.1 -> 24.4 mm, vias 9 -> 17
- net 9V: track 24.1 -> 18.1 mm, vias 20 -> 23
- net Net-(U9-IN+): track 16.0 -> 17.8 mm
- net Net-(C16-Pad2): track 5.95 -> 4.87 mm
- net Net-(U9-IN-): track 6.74 -> 6.00 mm
- net /CS2: track 53.5 -> 52.9 mm
- added copper zone on F.Cu, net 4.5V
