File: Pre Amp Stage/Pre Amp Stage.kicad_pcb (KiCad board)
At the start: 4 copper layers, 76.2 x 40.6 mm, 39 parts, among them J1 NMJ6HFD2, J2 Conn_01x03, J3 Conn_01x03, J4 MINIFIT-2-VERT, J5 Conn_01x03, J6 Conn_01x03, J7 Conn_01x03, J8 MINIFIT-2-VERT, Q1 Q_NJFET_DSG, U1 TL071HIDBVR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

Commit message: Added top copper gnd layer on pre amp
Routing:
- added copper zone on F.Cu, net GND
Changed lines of the file:
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@@
+	)
+	(zone
+		(net 1)
+		(net_name "GND")
+		(layer "F.Cu")
+		(hatch edge 0.5)
+		(connect_pads
+			(clearance 0.5)
+		)
+		(min_thickness 0.25)
+		(filled_areas_thickness no)
+		(fill yes
+			(thermal_gap 0.5)
+			(thermal_bridge_width 0.5)
+		)
+		(polygon
+			(pts
+				(xy 19.3294 22.2758) (xy 19.4056 68.0974) (xy 105.7402 68.0974) (xy 105.8672 22.4028)
+			)
+		)
 	)
 	(zone

Commit message: Incorporated changes from demo
Parts:
- added C12: 220p, Resistor_SMD:R_0603_1608Metric, F.Cu at (50.4, 57.0)
- added C13: 1u, Resistor_SMD:R_0603_1608Metric, F.Cu at (44.8, 57.6)
- added C14: 1u, Resistor_SMD:R_0603_1608Metric, F.Cu at (47.9, 51.6)
- added C15: 100u, Resistor_SMD:R_0805_2012Metric_Pad1.20x1.40mm_HandSolder, F.Cu at (89.2, 37.5)
- added U4: TL071HIDBVR, GTSR_KiCAD_Footprints:TL071, F.Cu at (47.4, 54.8)
- moved J8 5.51 mm to (93.7, 33.0)
- moved R2 3.62 mm to (62.5, 55.2)
- moved C1 3.02 mm to (50.4, 53.3)
- moved C2 3.02 mm to (50.4, 55.2)
- moved R1 2.38 mm to (52.9, 54.4)
- moved Q1 1.58 mm to (56.1, 52.7)
- moved C11 1.56 mm to (91.9, 41.5)
- moved C3 1.51 mm to (60.5, 52.1)
- moved R3 1.51 mm to (63.8, 52.1)
Connections:
- C1 pad 1: Net-(C1-Pad1) -> Net-(U4-IN-)
- C2 pad 1: Net-(C1-Pad1) -> Net-(U4-IN-)
- J1 pad T: Net-(C1-Pad1) -> Net-(U4-IN+)
- J8 pad 2: Net-(U3-OUT) -> Net-(C15-Pad2)
Routing:
- net Net-(U4-IN-): track 0.00 -> 9.51 mm
- net Net-(C1-Pad1): track 7.46 -> 0.00 mm
- net -15V: track 4.93 -> 9.69 mm, vias 2 -> 3
- net Net-(C15-Pad2): track 0.00 -> 4.50 mm
- net Net-(U4-IN+): track 0.00 -> 4.41 mm
- net GND: track 14.1 -> 18.1 mm, vias 8 -> 11
- net Net-(U3-OUT): track 47.2 -> 44.1 mm
- net +15V: track 5.86 -> 7.70 mm, vias 3 -> 4
- net Net-(Q1-S): track 4.46 -> 6.14 mm
