File: Pre Amp Stage/Pre Amp Stage.kicad_sch (KiCad schematic)
At the start: 38 parts, among them J1 NMJ6HFD2, J2 Conn_01x03, J3 Conn_01x03, J4 MINIFIT-2-VERT, J5 Conn_01x03, J6 Conn_01x03, J7 Conn_01x03, J8 MINIFIT-2-VERT, Q1 Q_NJFET_DSG, U1 TL071HIDBVR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

Commit message: Incorporated changes from demo
Parts:
- added C12: 220p, Resistor_SMD:R_0603_1608Metric, symbol Device:C
- added C13, C14: 1u, Resistor_SMD:R_0603_1608Metric, symbol Device:C
- added C15: 100u, Resistor_SMD:R_0805_2012Metric_Pad1.20x1.40mm_HandSolder, symbol Device:C
- added U4: TL071HIDBVR, GTSR_KiCAD_Footprints:TL071, symbol TL071HIDBVR:TL071HIDBVR
Connections:
- net +15V: now also C13.1, U4.5 (V+)
- net -15V: now also C14.1, U4.2 (V-)
- net GND: now also C12.2, C13.2, C14.2
- net at R7.2, R8.2, R9.2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: now also C15.1; no longer J8.2
- net at C1.1, C2.1: now also U4.1 (OUT), U4.4 (IN-); no longer J1.T
- net at C2.2, Q1.3 (G), R1.1: now also C12.1
- new net: C15.2, J8.2
- new net: J1.T, U4.3 (IN+)
Other:
- moved on the sheet: C7, J1, J4, J8, U2
