File: Power Amp Stage/Power Amp Board/Power Amp Board.kicad_pcb (KiCad board)
At the start: 4 copper layers, 103.6 x 60.6 mm, 31 parts, among them J2 Conn_01x02, J3 Conn_01x02, Q1 BC549, Q2 BC559, Q3 MJ15004, Q4 MJ15003, Q5 MJ15004, Q6 MJ15003, U1 ADA4522-2ARMZ-R7

Commit message: just absolutely lapped kyle
get fucked kyle
Parts:
- added U2: ADA4522-2ARMZ-R7, GTSR_KiCAD_Footprints:RM-8_ADI, F.Cu at (133.8, 86.6)
- moved C3 5.83 mm to (138.0, 86.4)
- moved C1 4.06 mm to (137.0, 92.5)
- moved C2 4.06 mm to (137.0, 103.1)
- moved R1 4.06 mm to (125.2, 89.5)
- moved R5 4.06 mm to (129.4, 92.5)
- moved R6 4.06 mm to (129.4, 103.1)
- moved R3 4.06 mm to (123.0, 98.5)
- moved R4 4.06 mm to (127.2, 93.9)
- moved D1 4.06 mm to (129.4, 95.7)
- moved D2 4.06 mm to (129.4, 99.9)
- moved Q1 4.06 mm to (132.9, 92.5)
- moved Q2 4.06 mm to (133.6, 103.1)
- moved R2 4.06 mm to (120.4, 93.9)
- moved R7 4.06 mm to (137.0, 95.9)
- moved R8 4.06 mm to (137.0, 99.7)
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Connections:
- C3 pad 2: Net-(P1-H) -> Net-(U2-INA+)
- P1 pad 1: Net-(P1-H) -> /buffer
Routing:
- net /buffer: track 0.00 -> 10.2 mm
- net Net-(P1-H): track 7.30 -> 0.00 mm
- net Net-(U2-INA+): track 0.00 -> 4.76 mm
- net Net-(Q2-C): track 85.5 -> 82.1 mm
- net /audio_in+: track 8.35 -> 5.07 mm
- net Net-(Q1-C): track 74.2 -> 76.9 mm
- net /post_pot: track 7.60 -> 10.2 mm
- net -24V: track 11.0 -> 13.1 mm, vias 20 -> 21
- net 24V: track 10.6 -> 12.3 mm, vias 20 -> 21
- net GND: vias 22 -> 23
