File: Power Amp Stage/Power Amp Board/Power Amp Board.kicad_pcb (KiCad board)
At the start: 4 copper layers, 103.6 x 60.6 mm, 32 parts, among them J2 Conn_01x02, J3 Conn_01x02, Q1 BC549, Q2 BC559, Q3 MJ15004, Q4 MJ15003, Q5 MJ15004, Q6 MJ15003, U1 ADA4522-2ARMZ-R7, U2 ADA4522-2ARMZ-R7

Commit message: fixed board again
Parts:
- R1, R3: value R -> 100k
- R10, R11, R12, R9: value R_US -> 4.7
- R2, R4, R5, R6: value R -> 10k
- R7, R8: value R -> 100
- moved J3 74.3 mm to (217.4, 98.0), turned to -90 degrees
- moved R9 37.9 mm to (152.0, 75.6), turned to -43 degrees
- moved R11 35.6 mm to (153.2, 120.0), turned to -134 degrees
- moved R10 28.1 mm to (188.2, 75.6), turned to -43 degrees
- moved R12 26.2 mm to (190.2, 120.0), turned to -134 degrees
- moved J1 11.4 mm to (132.2, 123.3), turned to 180 degrees
- moved C5 8.90 mm to (133.7, 110.2), turned to 180 degrees
- moved C4 8.57 mm to (125.3, 110.2), turned to 0 degrees
- moved R2 8.06 mm to (125.2, 87.4), turned to 180 degrees
- moved R4 7.96 mm to (123.0, 100.6), turned to 180 degrees
- moved P1 7.75 mm to (123.5, 75.8), turned to 0 degrees
- moved J2 6.45 mm to (140.0, 75.8), turned to 0 degrees
- moved Q3 4.02 mm to (163.3, 83.1), turned to -60 degrees
- moved Q5 4.02 mm to (199.1, 83.1), turned to -60 degrees
- moved Q4 3.76 mm to (166.8, 113.6), turned to 60 degrees
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Connections:
- J1 pad 1: 24V -> GND
- J1 pad 2: -24V -> GND
- J1 pad 3: GND -> 24V
- J1 pad 4: GND -> -24V
- J2 pad 1: /audio_in+ -> GND
- J2 pad 2: GND -> /audio_in+
- J3 pad 1: /audio_out+ -> GND
- J3 pad 2: GND -> /audio_out+
- P1 pad 1: /buffer -> GND
- P1 pad 2: /post_pot -> GND
- P1 pad 3: GND -> /post_pot
- P1 pad 4: GND -> /buffer
Routing:
- net /audio_out+: track 133.8 -> 236.2 mm
- net Net-(Q5-E): track 44.0 -> 6.25 mm
- net Net-(Q3-E): track 42.3 -> 6.73 mm
- net Net-(Q6-E): track 43.1 -> 7.73 mm
- net Net-(Q4-E): track 41.6 -> 9.01 mm
- net Net-(Q1-C): track 76.9 -> 80.9 mm
- net Net-(U1-INB-): track 7.96 -> 4.99 mm
- net Net-(U1-INA-): track 7.33 -> 4.54 mm
- net Net-(Q2-C): track 82.1 -> 84.2 mm
- net GND: track 1.42 -> 0.00 mm, vias 23 -> 49
- net -24V: vias 21 -> 41
- net 24V: vias 21 -> 41
- added copper zone on F.Cu, net /audio_out+
