File: phase90/phase90/phase90.kicad_pcb (KiCad board)
At the start: 4 copper layers, 55.4 x 32 mm, 65 parts, among them J1 Conn_02x08_Odd_Even, Q1 Q_NJFET_DSG, Q2 Q_NJFET_DSG, Q3 Q_NJFET_DSG, Q4 Q_NJFET_DSG, U1 TL071HIDBVR, U10 TL071HIDBVR, U11 TL071HIDBVR, U12 AD5290, U2 TL071HIDBVR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

Commit message: fixed connector also?
Connections:
- J1 pad 10: /GUITAR_OUT -> /GUITAR_IN
- J1 pad 11: /CS0 -> GND
- J1 pad 12: /MOSI -> GND
- J1 pad 3: GND -> unconnected-(J1-Pin_3-Pad3)
- J1 pad 4: GND -> unconnected-(J1-Pin_4-Pad4)
- J1 pad 6: /SPI_CLK -> /CS0
- J1 pad 7: unconnected-(J1-Pin_7-Pad7) -> /MOSI
- J1 pad 8: /GUITAR_IN -> /SPI_CLK
- J1 pad 9: unconnected-(J1-Pin_9-Pad9) -> /GUITAR_OUT
Routing:
- net /CS0: track 43.8 -> 53.5 mm, vias 2 -> 1
- net /SPI_CLK: track 55.1 -> 51.7 mm
- net /GUITAR_IN: track 62.3 -> 65.2 mm
- net /GUITAR_OUT: track 12.7 -> 10.2 mm
Changed lines of the file:
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@@
 	(net 16 "GND")
 	(net 17 "/SPI_CLK")
-	(net 18 "unconnected-(J1-Pin_9-Pad9)")
+	(net 18 "unconnected-(J1-Pin_3-Pad3)")
 	(net 19 "unconnected-(J1-Pin_5-Pad5)")
 	(net 20 "/CS0")
@@
 	(net 40 "Net-(U11-IN-)")
 	(net 41 "unconnected-(U12-SDO-Pad8)")
-	(net 42 "unconnected-(J1-Pin_7-Pad7)")
+	(net 42 "unconnected-(J1-Pin_4-Pad4)")
 	(net 43 "unconnected-(J1-Pin_16-Pad16)")
 	(net 44 "unconnected-(J1-Pin_15-Pad15)")
@@
 			(layers "*.Cu" "*.Mask")
 			(remove_unused_layers no)
-			(net 16 "GND")
+			(net 18 "unconnected-(J1-Pin_3-Pad3)")
 			(pinfunction "Pin_3")
-			(pintype "passive")
+			(pintype "passive+no_connect")
 		)
 		(pad "4" thru_hole circle
@@
 			(layers "*.Cu" "*.Mask")
 			(remove_unused_layers no)
-			(net 16 "GND")
+			(net 42 "unconnected-(J1-Pin_4-Pad4)")
 			(pinfunction "Pin_4")
-			(pintype "passive")
+			(pintype "passive+no_connect")
 		)
 		(pad "5" thru_hole circle
@@
 			(layers "*.Cu" "*.Mask")
 			(remove_unused_layers no)
-			(net 17 "/SPI_CLK")
+			(net 20 "/CS0")
 			(pinfunction "Pin_6")
 			(pintype "passive")
@@
 			(layers "*.Cu" "*.Mask")
 			(remove_unused_layers no)
-			(net 42 "unconnected-(J1-Pin_7-Pad7)")
+			(net 14 "/MOSI")
 			(pinfunction "Pin_7")
-			(pintype "passive+no_connect")
+			(pintype "passive")
+			(clearance 0.1)
 		)
 		(pad "8" thru_hole circle
@@
 			(layers "*.Cu" "*.Mask")
 			(remove_unused_layers no)
-			(net 5 "/GUITAR_IN")
+			(net 17 "/SPI_CLK")
 			(pinfunction "Pin_8")
 			(pintype "passive")
@@
 			(layers "*.Cu" "*.Mask")
 			(remove_unused_layers no)
-			(net 18 "unconnected-(J1-Pin_9-Pad9)")
+			(net 12 "/GUITAR_OUT")
 			(pinfunction "Pin_9")
-			(pintype "passive+no_connect")
+			(pintype "passive")
 		)
 		(pad "10" thru_hole circle
@@
 			(layers "*.Cu" "*.Mask")
 			(remove_unused_layers no)
-			(net 12 "/GUITAR_OUT")
+			(net 5 "/GUITAR_IN")
 			(pinfunction "Pin_10")
 			(pintype "passive")
@@
 			(layers "*.Cu" "*.Mask")
 			(remove_unused_layers no)
-			(net 20 "/CS0")
+			(net 16 "GND")
 			(pinfunction "Pin_11")
 			(pintype "passive")
@@
 			(layers "*.Cu" "*.Mask")
 			(remove_unused_layers no)
-			(net 14 "/MOSI")
+			(net 16 "GND")
 			(pinfunction "Pin_12")
 			(pintype "passive")
@@
 	)
 	(segment
-		(start 130.311 93.441)
-		(end 128.541818 93.441)
-		(width 0.4)
+		(start 83.072619 83.727381)
+		(end 83.072619 84.2)
+		(width 0.3)
 		(layer "F.Cu")
 		(net 5)
 	)
 	(segment
-		(start 126.8 91.699182)
+		(start 126.8 94.8)
 		(end 126.8 82.4)
-		(width 0.4)
-		(layer "F.Cu")
-		(net 5)
-	)
-	(segment
-		(start 83.072619 83.727381)
-		(end 83.072619 84.2)
-		(width 0.4)
+		(width 0.3)
 		(layer "F.Cu")
 		(net 5)
@@
 		(start 115.4 82.425)
 		(end 115.4 82.2)
-		(width 0.4)
+		(width 0.3)
 		(layer "F.Cu")
 		(net 5)
@@
 		(start 126.8 82.4)
 		(end 125.8 81.4)
-		(width 0.4)
+		(width 0.3)
+		(layer "F.Cu")
+		(net 5)
+	)
+	(segment
+		(start 125.8 81.4)
+		(end 116.2 81.4)
+		(width 0.3)
 		(layer "F.Cu")
 		(net 5)
@@
 		(start 115.4 82.2)
 		(end 116.2 81.4)
-		(width 0.4)
+		(width 0.3)
 		(layer "F.Cu")
 		(net 5)
 	)
 	(segment
-		(start 128.541818 93.441)
-		(end 126.8 91.699182)
-		(width 0.4)
+		(start 130.299 95.969)
+		(end 127.969 95.969)
+		(width 0.3)
 		(layer "F.Cu")
 		(net 5)
 	)
 	(segment
-		(start 131.6 94.73)
-		(end 130.311 93.441)
-		(width 0.4)
+		(start 127.969 95.969)
+		(end 126.8 94.8)
+		(width 0.3)
 		(layer "F.Cu")
 		(net 5)
 	)
 	(segment
-		(start 125.8 81.4)
-		(end 116.2 81.4)
-		(width 0.4)
+		(start 131.6 97.27)
+		(end 130.299 95.969)
+		(width 0.3)
 		(layer "F.Cu")
 		(net 5)
@@
 		(start 85.4 81.4)
 		(end 83.072619 83.727381)
-		(width 0.4)
+		(width 0.3)
 		(layer "F.Cu")
 		(net 5)
@@
 		(start 116.2 81.4)
 		(end 85.4 81.4)
-		(width 0.4)
+		(width 0.3)
 		(layer "F.Cu")
 		(net 5)
@@
 	)
 	(segment
-		(start 130.349 96.019)
-		(end 131.6 97.27)
-		(width 0.4)
+		(start 128.99 97.2)
+		(end 121.828618 97.2)
+		(width 0.3)
 		(layer "F.Cu")
 		(net 12)
 	)
 	(segment
-		(start 119.783618 95.155)
-		(end 120.647618 96.019)
-		(width 0.4)
+		(start 129.06 97.27)
+		(end 128.99 97.2)
+		(width 0.3)
 		(layer "F.Cu")
 		(net 12)
 	)
 	(segment
-		(start 120.647618 96.019)
-		(end 130.349 96.019)
-		(width 0.4)
+		(start 121.828618 97.2)
+		(end 119.783618 95.155)
+		(width 0.3)
 		(layer "F.Cu")
 		(net 12)
@@
 	)
 	(segment
-		(start 90.6 108.2)
-		(end 103 108.2)
+		(start 126.791 97.905389)
+		(end 123.735389 100.961)
+		(width 0.2)
+		(layer "B.Cu")
+		(net 14)
+	)
+	(segment
+		(start 129.06 94.73)
+		(end 126.791 96.999)
 		(width 0.2)
 		(layer "B.Cu")
@@
 	(segment
 		(start 110.239 100.961)
-		(end 130.449 100.961)
+		(end 103 108.2)
 		(width 0.2)
 		(layer "B.Cu")
@@
 	(segment
 		(start 103 108.2)
-		(end 110.239 100.961)
+		(end 90.6 108.2)
 		(width 0.2)
 		(layer "B.Cu")
@@
 	)
 	(segment
-		(start 130.449 100.961)
-		(end 131.6 99.81)
+		(start 126.791 96.999)
+		(end 126.791 97.905389)
+		(width 0.2)
+		(layer "B.Cu")
+		(net 14)
+	)
+	(segment
+		(start 123.735389 100.961)
+		(end 110.239 100.961)
 		(width 0.2)
 		(layer "B.Cu")
@@
 	)
 	(segment
-		(start 131.89776 98.6)
-		(end 132.751 97.74676)
+		(start 92.151 107.649)
+		(end 92.8 107)
 		(width 0.2)
 		(layer "B.Cu")
@@
 	)
 	(segment
-		(start 92.151 107.649)
-		(end 92.8 107)
+		(start 123.69 100.51)
+		(end 126.44 97.76)
 		(width 0.2)
 		(layer "B.Cu")
@@
 	)
 	(segment
-		(start 89.365952 108.234048)
-		(end 89.951 107.649)
+		(start 126.44 95.16)
+		(end 128.089934 93.510066)
 		(width 0.2)
 		(layer "B.Cu")
@@
 	)
 	(segment
-		(start 110.0729 100.56)
-		(end 126.44 100.56)
+		(start 103.6329 107)
+		(end 110.1229 100.51)
 		(width 0.2)
 		(layer "B.Cu")
@@
 	)
 	(segment
-		(start 103.6329 107)
-		(end 110.0729 100.56)
+		(start 128.089934 93.510066)
+		(end 130.380066 93.510066)
 		(width 0.2)
 		(layer "B.Cu")
@@
 	)
 	(segment
-		(start 132.751 97.74676)
-		(end 132.751 93.341)
+		(start 92.8 107)
+		(end 103.6329 107)
 		(width 0.2)
 		(layer "B.Cu")
@@
 	)
 	(segment
-		(start 89.951 107.649)
-		(end 92.151 107.649)
+		(start 130.380066 93.510066)
+		(end 131.6 94.73)
 		(width 0.2)
 		(layer "B.Cu")
@@
 	)
 	(segment
-		(start 92.8 107)
-		(end 103.6329 107)
+		(start 126.44 97.76)
+		(end 126.44 95.16)
 		(width 0.2)
 		(layer "B.Cu")
@@
 	)
 	(segment
-		(start 128.4 98.6)
-		(end 131.89776 98.6)
+		(start 89.951 107.649)
+		(end 92.151 107.649)
 		(width 0.2)
 		(layer "B.Cu")
@@
 	)
 	(segment
-		(start 126.44 100.56)
-		(end 128.4 98.6)
+		(start 110.1229 100.51)
+		(end 123.69 100.51)
 		(width 0.2)
 		(layer "B.Cu")
@@
 	)
 	(segment
-		(start 132.751 93.341)
-		(end 131.6 92.19)
+		(start 89.365952 108.234048)
+		(end 89.951 107.649)
 		(width 0.2)
 		(layer "B.Cu")
@@
 	)
 	(segment
-		(start 129.06 99.81)
-		(end 126.01 99.81)
-		(width 0.2)
-		(layer "F.Cu")
-		(net 20)
-	)
-	(segment
 		(start 90 106.8)
 		(end 89.8 106.8)
@@
 		(net 20)
 	)
-	(segment
-		(start 126.01 99.81)
-		(end 126 99.8)
-		(width 0.2)
-		(layer "F.Cu")
-		(net 20)
-	)
 	(via
 		(at 90 106.8)
@@
 		(net 20)
 	)
-	(via
-		(at 126 99.8)
-		(size 0.6)
-		(drill 0.3)
-		(layers "F.Cu" "B.Cu")
+	(segment
+		(start 90.910132 106.8)
+		(end 90 106.8)
+		(width 0.2)
+		(layer "B.Cu")
+		(net 20)
+	)
+	(segment
+		(start 126 92.6)
+		(end 126 97.6)
+		(width 0.2)
+		(layer "B.Cu")
 		(net 20)
 	)
@@
 	)
 	(segment
-		(start 125.641 100.159)
+		(start 127.685588 90.914412)
+		(end 126 92.6)
+		(width 0.2)
+		(layer "B.Cu")
+		(net 20)
+	)
+	(segment
+		(start 123.441 100.159)
 		(end 108.654701 100.159)
 		(width 0.2)
@@
 	)
 	(segment
-		(start 126 99.8)
-		(end 125.641 100.159)
+		(start 126 97.6)
+		(end 123.441 100.159)
+		(width 0.2)
+		(layer "B.Cu")
+		(net 20)
+	)
+	(segment
+		(start 131.6 92.19)
+		(end 130.324412 90.914412)
 		(width 0.2)
 		(layer "B.Cu")
@@
 	)
 	(segment
-		(start 90.910132 106.8)
-		(end 90 106.8)
+		(start 130.324412 90.914412)
+		(end 127.685588 90.914412)
 		(width 0.2)
 		(layer "B.Cu")

Commit message: added buffers and caps for op-amps on effect boards
Parts:
- added C10: 1u, Capacitor_SMD:C_0603_1608Metric, B.Cu at (100.8, 91.0)
- added C11: 1u, Capacitor_SMD:C_0603_1608Metric, B.Cu at (109.8, 91.0)
- added C12: 1u, Capacitor_SMD:C_0603_1608Metric, B.Cu at (107.0, 108.0)
- added C13: 1u, Capacitor_SMD:C_0603_1608Metric, B.Cu at (113.0, 106.8)
- added C14: 1u, Capacitor_SMD:C_0603_1608Metric, B.Cu at (118.8, 108.0)
- added C15: 1u, Capacitor_SMD:C_0603_1608Metric, B.Cu at (82.0, 88.8)
- added C16: 1u, Capacitor_SMD:C_0603_1608Metric, B.Cu at (117.8, 91.0)
- added C17: 1u, Capacitor_SMD:C_0603_1608Metric, B.Cu at (124.0, 91.8)
- added C18: 1u, Capacitor_SMD:C_0603_1608Metric, B.Cu at (95.8, 110.0)
- added C3: 1u, Capacitor_SMD:C_0603_1608Metric, B.Cu at (92.8, 91.0)
- added U3: TL071HIDBVR, Package_TO_SOT_SMD:SOT-23-5, F.Cu at (81.2, 85.0)
- moved C5 3.83 mm to (86.0, 83.2), turned to -90 degrees
- moved R3 3.60 mm to (78.8, 89.8)
- moved R1 3.60 mm to (78.8, 92.0)
- moved R2 3.60 mm to (78.8, 94.2)
- moved C4 1.62 mm to (82.8, 88.0)
- moved R15 1.55 mm to (83.0, 90.0)
Connections:
- C4 pad 1: 6V -> Net-(U3-IN-)
- R15 pad 1: 6V -> Net-(U3-IN-)
Routing:
- net 12V: track 22.8 -> 43.6 mm, vias 18 -> 20
- net 6V: track 6.60 -> 16.5 mm
- net Net-(U3-IN-): track 0.00 -> 7.32 mm
- net /GUITAR_IN: track 65.2 -> 60.0 mm
- net GND: track 26.9 -> 28.5 mm, vias 30 -> 31
Other:
- board size 55.4 x 32 mm -> 58.4 x 32 mm

Commit message: fixes for Marco's dr
Parts:
- moved R1 11.2 mm to (81.0, 103.0)
- moved R2 11.2 mm to (81.0, 105.2)
- moved R3 11.2 mm to (81.0, 100.8)
- moved U3 9.05 mm to (81.2, 94.0), turned to -90 degrees
- moved C5 5.75 mm to (81.0, 86.0), turned to 180 degrees
- moved R15 1.23 mm to (81.8, 90.0)
- moved C4 1.00 mm to (81.8, 88.0)
Routing:
- net /GUITAR_IN: track 60.0 -> 65.7 mm
- net Net-(U3-IN-): track 7.32 -> 9.02 mm
- net Net-(Q1-D): track 15.5 -> 17.1 mm
- net Net-(U7-IN-): track 4.37 -> 5.31 mm
- net 6V: track 16.5 -> 17.3 mm
- net GND: track 28.5 -> 29.2 mm
- net 12V: track 43.6 -> 44.1 mm, vias 20 -> 21
