File: Digital and Recording Board/digital_and_recording/digital_and_recording.kicad_pcb (KiCad board)
At the start: 4 copper layers, 47 x 106.3 mm, 42 parts, among them J1 Headphones, J2 Screen, J3 USB_Breakout, J4 Joystick, J6 MINIFIT-2-VERT, J7 MINIFIT-2-VERT, J8 MINIFIT-2-VERT, U1 Daisy_Seed, U2 Daisy_Seed_Recording, U3 Bypass 2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

Commit message: fixed usb pitch issue
Parts:
- J1: footprint footprints:CONN_SD-5566-002_02_MOL -> Kyle's Footprints:CONN_SD-5566-002_02_MOL
- J3: footprint Connector_PinHeader_1.00mm:PinHeader_1x04_P1.00mm_Vertical -> Connector_PinHeader_2.54mm:PinHeader_1x04_P2.54mm_Vertical
- moved J3 2.66 mm to (160.4, 113.6)
Routing:
- net /Connectors/USB_D-: track 51.9 -> 51.2 mm
Changed lines of the file:
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@@
 		(embedded_fonts no)
 	)
-	(footprint "Connector_PinHeader_1.00mm:PinHeader_1x04_P1.00mm_Vertical"
+	(footprint "Connector_PinHeader_2.54mm:PinHeader_1x04_P2.54mm_Vertical"
 		(layer "F.Cu")
-		(at 157.75 113.75 -90)
-		(descr "Through hole straight pin header, 1x04, 1.00mm pitch, single row")
-		(tags "Through hole pin header THT 1x04 1.00mm single row")
+		(at 160.41 113.6 -90)
+		(descr "Through hole straight pin header, 1x04, 2.54mm pitch, single row")
+		(tags "Through hole pin header THT 1x04 2.54mm single row")
 		(property "Reference" "J3"
-			(at 0 -2 90)
+			(at -2.6 -0.19 0)
 			(layer "F.SilkS")
 			(effects
@@
 		)
 		(property "Value" "USB_Breakout"
-			(at 2.5 1.5 0)
+			(at 0 10 270)
 			(layer "F.Fab")
 			(effects
@@
 		)
 		(property "Datasheet" "~"
-			(at 0 0 90)
+			(at 0 0 270)
 			(layer "F.Fab")
 			(hide yes)
@@
 		)
 		(property "Description" "Generic connector, single row, 01x04, script generated (kicad-library-utils/schlib/autogen/connector/)"
-			(at 0 0 90)
+			(at 0 0 270)
 			(layer "F.Fab")
 			(hide yes)
@@
 		(attr through_hole)
 		(fp_line
-			(start -0.745 3.61)
-			(end -0.41003 3.61)
+			(start -1.38 9)
+			(end 1.38 9)
 			(stroke
 				(width 0.12)
@@
 		)
 		(fp_line
-			(start 0.41003 3.61)
-			(end 0.745 3.61)
+			(start -1.38 1.27)
+			(end -1.38 9)
 			(stroke
 				(width 0.12)
@@
 		)
 		(fp_line
-			(start -0.745 0.735)
-			(end -0.745 3.61)
+			(start -1.38 1.27)
+			(end 1.38 1.27)
 			(stroke
 				(width 0.12)
@@
 		)
 		(fp_line
-			(start -0.745 0.735)
-			(end -0.685565 0.735)
+			(start 1.38 1.27)
+			(end 1.38 9)
 			(stroke
 				(width 0.12)
@@
 		)
 		(fp_line
-			(start 0.685565 0.735)
-			(end 0.745 0.735)
+			(start -1.38 0)
+			(end -1.38 -1.38)
 			(stroke
 				(width 0.12)
@@
 		)
 		(fp_line
-			(start 0.745 0.735)
-			(end 0.745 3.61)
+			(start -1.38 -1.38)
+			(end 0 -1.38)
 			(stroke
 				(width 0.12)
@@
 		)
 		(fp_line
-			(start -0.745 0)
-			(end -0.745 -0.735)
-			(stroke
-				(width 0.12)
-				(type solid)
-			)
-			(layer "F.SilkS")
-		)
-		(fp_line
-			(start -0.745 -0.735)
-			(end 0 -0.735)
-			(stroke
-				(width 0.12)
-				(type solid)
-			)
-			(layer "F.SilkS")
-		)
-		(fp_line
-			(start -1.14 4)
-			(end 1.14 4)
+			(start -1.77 9.39)
+			(end 1.77 9.39)
 			(stroke
 				(width 0.05)
@@
 		)
 		(fp_line
-			(start 1.14 4)
-			(end 1.14 -1)
+			(start 1.77 9.39)
+			(end 1.77 -1.77)
 			(stroke
 				(width 0.05)
@@
 		)
 		(fp_line
-			(start -1.14 -1)
-			(end -1.14 4)
+			(start -1.77 -1.77)
+			(end -1.77 9.39)
 			(stroke
 				(width 0.05)
@@
 		)
 		(fp_line
-			(start 1.14 -1)
-			(end -1.14 -1)
+			(start 1.77 -1.77)
+			(end -1.77 -1.77)
 			(stroke
 				(width 0.05)
@@
 		)
 		(fp_line
-			(start -0.635 3.5)
-			(end -0.635 -0.1825)
+			(start -1.27 8.89)
+			(end -1.27 -0.635)
 			(stroke
 				(width 0.1)
@@
 		)
 		(fp_line
-			(start 0.635 3.5)
-			(end -0.635 3.5)
+			(start 1.27 8.89)
+			(end -1.27 8.89)
 			(stroke
 				(width 0.1)
@@
 		)
 		(fp_line
-			(start -0.635 -0.1825)
-			(end -0.3175 -0.5)
+			(start -1.27 -0.635)
+			(end -0.635 -1.27)
 			(stroke
 				(width 0.1)
@@
 		)
 		(fp_line
-			(start -0.3175 -0.5)
-			(end 0.635 -0.5)
+			(start -0.635 -1.27)
+			(end 1.27 -1.27)
 			(stroke
 				(width 0.1)
@@
 		)
 		(fp_line
-			(start 0.635 -0.5)
-			(end 0.635 3.5)
+			(start 1.27 -1.27)
+			(end 1.27 8.89)
 			(stroke
 				(width 0.1)
@@
 		)
 		(fp_text user "${REFERENCE}"
-			(at 0 1.5 0)
+			(at 0 3.81 0)
 			(layer "F.Fab")
 			(effects
 				(font
-					(size 0.76 0.76)
-					(thickness 0.114)
+					(size 1 1)
+					(thickness 0.15)
 				)
 			)
@@
 		(pad "1" thru_hole rect
 			(at 0 0 270)
-			(size 0.85 0.85)
-			(drill 0.5)
+			(size 1.7 1.7)
+			(drill 1)
 			(layers "*.Cu" "*.Mask")
 			(remove_unused_layers no)
@@
 		)
 		(pad "2" thru_hole circle
-			(at 0 1 270)
-			(size 0.85 0.85)
-			(drill 0.5)
+			(at 0 2.54 270)
+			(size 1.7 1.7)
+			(drill 1)
 			(layers "*.Cu" "*.Mask")
 			(remove_unused_layers no)
@@
 		)
 		(pad "3" thru_hole circle
-			(at 0 2 270)
-			(size 0.85 0.85)
-			(drill 0.5)
+			(at 0 5.08 270)
+			(size 1.7 1.7)
+			(drill 1)
 			(layers "*.Cu" "*.Mask")
 			(remove_unused_layers no)
@@
 		)
 		(pad "4" thru_hole circle
-			(at 0 3 270)
-			(size 0.85 0.85)
-			(drill 0.5)
+			(at 0 7.62 270)
+			(size 1.7 1.7)
+			(drill 1)
 			(layers "*.Cu" "*.Mask")
 			(remove_unused_layers no)
@@
 		)
 		(embedded_fonts no)
-		(model "${KICAD9_3DMODEL_DIR}/Connector_PinHeader_1.00mm.3dshapes/PinHeader_1x04_P1.00mm_Vertical.step"
+		(model "${KICAD9_3DMODEL_DIR}/Connector_PinHeader_2.54mm.3dshapes/PinHeader_1x04_P2.54mm_Vertical.step"
 			(offset
 				(xyz 0 0 0)
@@
 		(embedded_fonts no)
 	)
-	(footprint "footprints:CONN_SD-5566-002_02_MOL"
+	(footprint "Kyle's Footprints:CONN_SD-5566-002_02_MOL"
 		(layer "F.Cu")
 		(at 132.25 137 180)
@@
 	)
 	(segment
-		(start 155.75 113.75)
-		(end 155.75 112.5)
+		(start 155.75 113.18)
+		(end 155.33 113.6)
+		(width 0.2)
+		(layer "F.Cu")
+		(net 13)
+	)
+	(segment
+		(start 155.75 112.5)
+		(end 155.75 113.18)
 		(width 0.2)
 		(layer "F.Cu")
@@
 	(segment
 		(start 155.75 112.5)
-		(end 156.25 112)
+		(end 156.725 111.525)
 		(width 0.2)
 		(layer "F.Cu")
@@
 	)
 	(via
-		(at 156.25 112)
+		(at 156.725 111.525)
 		(size 0.5)
 		(drill 0.3)
@@
 	)
 	(segment
-		(start 162.25 75.25)
-		(end 162.25 106)
+		(start 162.25 106)
+		(end 162.25 75.25)
 		(width 0.2)
 		(layer "B.Cu")
@@
 	)
 	(segment
-		(start 170 67.5)
-		(end 162.25 75.25)
+		(start 156.725 111.525)
+		(end 162.25 106)
 		(width 0.2)
 		(layer "B.Cu")
@@
 	)
 	(segment
-		(start 162.25 106)
-		(end 156.25 112)
+		(start 162.25 75.25)
+		(end 170 67.5)
 		(width 0.2)
 		(layer "B.Cu")
@@
 	)
 	(segment
-		(start 156.75 112.5)
-		(end 157.25 112)
+		(start 157.87 113.6)
+		(end 157.87 111.93)
 		(width 0.2)
 		(layer "F.Cu")
@@
 	)
 	(segment
-		(start 170 69.25)
-		(end 171.02 68.23)
+		(start 157.87 111.93)
+		(end 158 111.8)
 		(width 0.2)
 		(layer "F.Cu")
@@
 	)
 	(segment
-		(start 171.02 68.23)
-		(end 171.45 68.23)
+		(start 170 69.25)
+		(end 171.02 68.23)
 		(width 0.2)
 		(layer "F.Cu")
@@
 	)
 	(segment
-		(start 156.75 113.75)
-		(end 156.75 112.5)
+		(start 171.02 68.23)
+		(end 171.45 68.23)
 		(width 0.2)
 		(layer "F.Cu")
@@
 	)
 	(via
-		(at 157.25 112)
+		(at 158 111.8)
 		(size 0.5)
 		(drill 0.3)
@@
 	)
 	(segment
-		(start 163 76.25)
-		(end 170 69.25)
+		(start 158 111.25)
+		(end 163 106.25)
 		(width 0.2)
 		(layer "B.Cu")
@@
 	)
 	(segment
-		(start 163 106.25)
-		(end 163 76.25)
+		(start 163 76.25)
+		(end 170 69.25)
 		(width 0.2)
 		(layer "B.Cu")
@@
 	)
 	(segment
-		(start 157.25 112)
-		(end 163 106.25)
+		(start 158 111.8)
+		(end 158 111.25)
 		(width 0.2)
 		(layer "B.Cu")
@@
 	)
 	(segment
-		(start 161.25 114.25)
-		(end 159.5 116)
+		(start 163 106.25)
+		(end 163 76.25)
 		(width 0.2)
 		(layer "B.Cu")
-		(net 15)
+		(net 14)
 	)
 	(segment
-		(start 148.5 114.25)
-		(end 148.5 91.184)
+		(start 148.5 91.184)
+		(end 145.836 88.52)
 		(width 0.2)
 		(layer "B.Cu")
@@
 	)
 	(segment
-		(start 159.5 116)
-		(end 150.25 116)
+		(start 148.5 114.25)
+		(end 148.5 91.184)
 		(width 0.2)
 		(layer "B.Cu")
@@
 	)
 	(segment
-		(start 148.5 91.184)
-		(end 145.836 88.52)
+		(start 161.4 116)
+		(end 150.25 116)
 		(width 0.2)
 		(layer "B.Cu")
@@
 	(segment
 		(start 167.1 114.25)
-		(end 161.25 114.25)
+		(end 163.15 114.25)
+		(width 0.2)
+		(layer "B.Cu")
+		(net 15)
+	)
+	(segment
+		(start 163.15 114.25)
+		(end 161.4 116)
 		(width 0.2)
 		(layer "B.Cu")
